File: BMS/BMS Board/BMS Board.kicad_pcb (KiCad board)
At the start: 2 copper layers, 175.3 x 92.1 mm, 234 parts, among them J1 10129379-904002BLF, J2 640456-3, K1 G5PZ-1A_DC12, M1 AO3402, M10 AO3402, M11 AO3402, M12 AO3402, M13 AO3402, M14 AO3402, M15 AO3402, M16 AO3402, M17 AO3402, M18 AO3402, M19 AO3402, M2 AO3402, M20 AO3402, M21 AO3402, M22 AO3402, M3 AO3402, M4 AO3402, M5 AO3402, M6 AO3402, M7 AO3402, M8 AO3402, M9 AO3402, P1 Power_Pad, P2 Power_Pad, P3 Power_Pad, P4 Power_Pad, P5 Power_Pad, P6 Power_Pad, Q1 STD12N60DM2AG, Q2 AO3402, U1 INA149AID, U10 INA149AID, U11 INA149AID, U12 INA149AID, U13 INA149AID, U14 INA149AID, U15 INA149AID, U16 INA149AID, U17 INA149AID, U18 INA149AID, U19 INA149AID, U2 INA149AID, U20 INA149AID, U21 TMP235AEDBZTQ1, U22 TMP235AEDBZTQ1, U23 TMP235AEDBZTQ1, U24 TMP235AEDBZTQ1, U25 ADS1248IPWR, U26 ADS1248IPWR, U27 ADS1248IPWR, U28 MAX6225ACSA+, U29 MCP23008-E_SO, U3 INA149AID, U30 MCP23008-E_SO, U31 MCP23008-E_SO, U4 INA149AID, U5 INA149AID, U6 INA149AID, U7 INA149AID, U8 INA149AID, U9 INA149AID

Commit message: changed ui components to be classes instead of methods in Screen class
Parts:
- removed O21: TLP2270_TP4,E, SamacSys_Parts:SOIC127P1105X220-8N
- removed the R116 at (279.4, 417.5)
- added C17: 0805ZC104MAT2A, SamacSys_Parts:CAPC2012X94N, F.Cu at (271.8, 408.6)
- added D1: S1G, SamacSys_Parts:DIOM5227X250N, F.Cu at (268.9, 361.9)
- added D2: S1G, SamacSys_Parts:DIOM5227X250N, F.Cu at (251.8, 373.1)
- added IC1: TLP2310_TPL,E, SamacSys_Parts:SOIC127P700X220-6N, F.Cu at (278.1, 414.7)
- added IC2: TLP2310_TPL,E, SamacSys_Parts:SOIC127P700X220-6N, F.Cu at (273.4, 414.7)
- added R102: ERJ-S06F2002V, SamacSys_Parts:RESC2012X70N, F.Cu at (269.6, 406.7)
- added R105: ERJ-S06J472V, SamacSys_Parts:RESC2012X70N, F.Cu at (220.0, 350.5)
- added R106: ERJ-S06J472V, SamacSys_Parts:RESC2012X70N, F.Cu at (218.1, 350.5)
- added R107: ERJ-S06J472V, SamacSys_Parts:RESC2012X70N, F.Cu at (216.2, 353.4)
- added R108: ERJ-S06J472V, SamacSys_Parts:RESC2012X70N, F.Cu at (216.2, 355.3)
- added R111: ERJ-S06J472V, SamacSys_Parts:RESC2012X70N, F.Cu at (218.1, 374.3)
- added R112: ERJ-S06J472V, SamacSys_Parts:RESC2012X70N, F.Cu at (216.9, 375.6)
- added R113: ERJ-S06J472V, SamacSys_Parts:RESC2012X70N, B.Cu at (211.5, 375.3)
- added R114: ERJ-S06J472V, SamacSys_Parts:RESC2012X70N, F.Cu at (215.9, 379.4)
- added R117: ERJ-S06J472V, SamacSys_Parts:RESC2012X70N, F.Cu at (218.4, 406.4)
- added R118: ERJ-S06J472V, SamacSys_Parts:RESC2012X70N, F.Cu at (217.8, 409.6)
- added R119: ERJ-S06J472V, SamacSys_Parts:RESC2012X70N, F.Cu at (216.5, 410.8)
- added R120: ERJ-S06J472V, SamacSys_Parts:RESC2012X70N, F.Cu at (215.9, 413.1)
- added R121: ERJ-S06J472V, SamacSys_Parts:RESC2012X70N, F.Cu at (216.2, 366.4)
- added R122: ERJ-S06J472V, SamacSys_Parts:RESC2012X70N, F.Cu at (215.3, 363.9)
- added R123: ERJ-S06J472V, SamacSys_Parts:RESC2012X70N, F.Cu at (218.8, 392.1)
- added R124: ERJ-S06J472V, SamacSys_Parts:RESC2012X70N, F.Cu at (216.2, 389.3)
- added R125: ERJ-S06J472V, SamacSys_Parts:RESC2012X70N, B.Cu at (215.3, 388.0)
- added R126: ERJ-S06J472V, SamacSys_Parts:RESC2012X70N, F.Cu at (215.6, 424.2)
- added R127: ERJ-S06J472V, SamacSys_Parts:RESC2012X70N, F.Cu at (215.6, 422.3)
- added R128: ERJ-S06J472V, SamacSys_Parts:RESC2012X70N, F.Cu at (215.6, 418.5)
- added R135: ERJ-P06F2200V, SamacSys_Parts:RESC2012X70N, F.Cu at (281.6, 408.3)
- C18: renamed from C17; moved to B.Cu
- moved R137 16.2 mm to (273.4, 421.0)
- moved R101 11.1 mm to (280.4, 386.4), turned to 90 degrees
- moved R136 4.51 mm to (279.4, 408.3)
- moved R138 3.49 mm to (269.9, 421.0)
- moved C18 2.62 mm to (278.1, 417.8), turned to 180 degrees
- moved LED1 2.42 mm to (281.6, 414.7), turned to 90 degrees
- moved LED2 0.95 mm to (269.9, 414.7)
- renumbered R102 to R103, R103 to R104, R104 to R109, R105 to R110, R106 to R115, R107 to R116, R108 to R129, R109 to R130, R110 to R131, R111 to R132, R112 to R133, R113 to R134, R114 to R136, R115 to R137, R117 to R138, R118 to R139, R119 to R140, R120 to R141, R121 to R142
Connections:
- net /Control/3v3 renamed /Communication/3v3
- C18 pad 2: GNDREF -> Net-(C18-Pad2)
- J1 pad 4: GNDREF -> Net-(C18-Pad2)
- LED2 pad 1: GNDREF -> Net-(C18-Pad2)
- R101 pad 2: GNDREF -> B-
- R137 pad 1: /Communication/RX -> Net-(IC2-Pad1)
- R137 pad 2: Net-(O21-Pad4) -> Net-(J1-Pad3)
- U25 pad 11: V19 -> Net-(R105-Pad2)
- U25 pad 12: V18 -> Net-(R106-Pad2)
- U25 pad 13: V17 -> Net-(R107-Pad2)
- U25 pad 14: V20 -> Net-(R108-Pad2)
- U25 pad 15: V16 -> Net-(R122-Pad1)
- U25 pad 16: V15 -> Net-(R121-Pad1)
- U26 pad 11: V13 -> Net-(R111-Pad2)
- U26 pad 12: V14 -> Net-(R112-Pad2)
- U26 pad 13: V11 -> Net-(R113-Pad2)
- U26 pad 14: V10 -> Net-(R114-Pad2)
- U26 pad 15: V9 -> Net-(R125-Pad1)
- U26 pad 16: V12 -> Net-(R124-Pad1)
- U26 pad 17: V8 -> Net-(R123-Pad1)
- U27 pad 11: V7 -> Net-(R117-Pad2)
- U27 pad 12: V5 -> Net-(R118-Pad2)
- U27 pad 13: V6 -> Net-(R119-Pad2)
- U27 pad 14: V3 -> Net-(R120-Pad2)
- U27 pad 15: V2 -> Net-(R128-Pad1)
- U27 pad 16: V1 -> Net-(R127-Pad1)
- U27 pad 17: V4 -> Net-(R126-Pad1)
Routing:
- net P-: track 0.00 -> 40.5 mm, vias 0 -> 1
- net Net-(C18-Pad2): track 0.00 -> 22.3 mm, vias 0 -> 2
- net /Communication/3v3: track 210.2 -> 227.5 mm
- net V11: track 15.6 -> 4.83 mm, vias 1 -> 0
- net Net-(D1-Pad1): track 0.00 -> 10.2 mm
- net V7: track 22.1 -> 12.4 mm
- net Net-(R113-Pad2): track 0.00 -> 9.09 mm, vias 0 -> 1
- net V18: track 23.1 -> 14.1 mm
- net V19: track 24.5 -> 16.0 mm
- net Net-(R117-Pad2): track 0.00 -> 7.86 mm
- net /Communication/RX: track 33.7 -> 41.5 mm, vias 0 -> 2
- net /Control/CELL_4: track 287.4 -> 294.7 mm
- net Net-(R106-Pad2): track 0.00 -> 7.14 mm
- net V8: track 24.2 -> 17.1 mm
- net Net-(D2-Pad2): track 2.69 -> 9.68 mm
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Other:
- board text added: "01 02"
- board text added: "03 04"
- board text added: "05 06"
- board text added: "07 08"
- board text added: "09 10"
- board text added: "11 12"
- board text added: "13 14"
- board text added: "15 16"
- board text added: "17 18"
- board text added: "19 20"
- board text added: "NC GND"

Commit message: "SingleDigitNumberSelector" now blinks when idle.
Parts:
- IC1, IC2: value TLP2310_TPL,E -> TLP2766A_TP,E; footprint SamacSys_Parts:SOIC127P700X220-6N -> SamacSys_Parts:SOT127P1000X230-6N
- moved R114 292.7 mm to (215.9, 122.6)
- moved R116 292.7 mm to (218.1, 122.6)
- moved C18 292.7 mm to (208.6, 122.9)
- moved IC1 291.5 mm to (214.6, 130.2)
- moved IC2 291.5 mm to (209.9, 130.2)
- moved LED1 291.5 mm to (218.1, 130.2)
- moved LED2 291.5 mm to (206.4, 130.2)
- moved C1 289.9 mm to (163.8, 141.6)
- moved C12 289.9 mm to (147.0, 128.0)
- moved C13 289.9 mm to (147.0, 137.2)
- moved C14 289.9 mm to (166.7, 136.8)
- moved C15 289.9 mm to (166.1, 133.3)
- moved C5 289.9 mm to (147.0, 68.6)
- moved C6 289.9 mm to (147.0, 81.0)
- moved C8 289.9 mm to (147.0, 92.4)
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- renumbered C18 to C17, C17 to C18, R103 to R102, R104 to R103, R109 to R104, R110 to R105, R115 to R106, R116 to R107, R129 to R108, R130 to R109, R131 to R110, R132 to R111, R133 to R112, R134 to R113, R136 to R114, R137 to R115, R135 to R116, R138 to R117, R139 to R118, R140 to R119, R141 to R120, R142 to R121, R102 to R122, R105 to R123, R106 to R124, R107 to R125, R108 to R126, R111 to R127, R112 to R128, R113 to R129, R114 to R130, R117 to R131, R118 to R132, R119 to R133, R120 to R134, R121 to R135, R122 to R136, R123 to R137, R124 to R138, R125 to R139, R126 to R140, R127 to R141, R128 to R142
Routing:
- net /Communication/RX: track 41.5 -> 38.4 mm
- net /Communication/3v3: track 227.5 -> 230.4 mm
- net /Communication/TX: track 38.9 -> 36.1 mm
- net Net-(LED2-Pad2): track 4.45 -> 5.90 mm
- net Net-(LED1-Pad2): track 4.45 -> 5.72 mm
- net Net-(C17-Pad1): track 8.77 -> 9.72 mm
- net Net-(C17-Pad2): track 22.3 -> 23.0 mm
- net GNDREF: vias 98 -> 99

Commit message: ...
Parts:
- added G***: LOGO, Logo:Logo, F.Cu at (180.3, 78.1)
- added LED3: HSMG-C170, SamacSys_Parts:LEDC2012X80N, F.Cu at (194.0, 82.9)
- added R143: ERJ-P06F2200V, SamacSys_Parts:RESC2012X70N, B.Cu at (199.1, 90.2)
- R114, R115: value ERJ-6ENF5600V -> ERJ-P06F2200V
Connections:
- U29 pad 5: /Communication/3v3 -> GNDREF
Routing:
- net Net-(LED3-Pad2): track 0.00 -> 8.99 mm, vias 0 -> 1
- net /Control/C_SIG: track 39.1 -> 42.6 mm
- net /Communication/3v3: track 230.4 -> 232.6 mm
Other:
- board text added: "- Adin Ackerman"
- board text added: "Battery Management System V2"
- board text added: "Relay"
- board text added: "Teo"
