File: BMS/BMS Board/Discharge.sch (KiCad schematic (older format))
At the start: 140 parts, among them M1 AO3402, M10 AO3402, M11 AO3402, M12 AO3402, M13 AO3402, M14 AO3402, M15 AO3402, M16 AO3402, M17 AO3402, M18 AO3402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

Commit message: workin on BMS also reset my computer so KiCad added some recovery files
Parts:
- M1, M10, M11, M12, M13, M14, M15, M16, M17, M18, M19, M2, M20, M3, M4, M5, M6, M7, M8, M9: symbol MOSFET:AO3402 -> BMS-Board-rescue:AO3402-MOSFET
Changed lines of the file:
@@
 $EndComp
 $Comp
-L MOSFET:AO3402 M20
+L BMS-Board-rescue:AO3402-MOSFET M20
 U 1 1 5E91C5D7
 P 12000 27900
+AR Path="/5E91C5D7" Ref="M20"  Part="1"
+AR Path="/5E8E2BA1/5E91C5D7" Ref="M20"  Part="1"
 F 0 "M20" H 12228 27946 50  0000 L CNN
 F 1 "AO3402" H 12228 27855 50  0000 L CNN
@@
 $EndComp
 $Comp
-L MOSFET:AO3402 M19
+L BMS-Board-rescue:AO3402-MOSFET M19
 U 1 1 5E97DB76
 P 12000 26700
+AR Path="/5E97DB76" Ref="M19"  Part="1"
+AR Path="/5E8E2BA1/5E97DB76" Ref="M19"  Part="1"
 F 0 "M19" H 12228 26746 50  0000 L CNN
 F 1 "AO3402" H 12228 26655 50  0000 L CNN
@@
 $EndComp
 $Comp
-L MOSFET:AO3402 M18
+L BMS-Board-rescue:AO3402-MOSFET M18
 U 1 1 5E991AA7
 P 12000 25500
+AR Path="/5E991AA7" Ref="M18"  Part="1"
+AR Path="/5E8E2BA1/5E991AA7" Ref="M18"  Part="1"
 F 0 "M18" H 12228 25546 50  0000 L CNN
 F 1 "AO3402" H 12228 25455 50  0000 L CNN
@@
 $EndComp
 $Comp
-L MOSFET:AO3402 M17
+L BMS-Board-rescue:AO3402-MOSFET M17
 U 1 1 5E99AE23
 P 12000 24300
+AR Path="/5E99AE23" Ref="M17"  Part="1"
+AR Path="/5E8E2BA1/5E99AE23" Ref="M17"  Part="1"
 F 0 "M17" H 12228 24346 50  0000 L CNN
 F 1 "AO3402" H 12228 24255 50  0000 L CNN
@@
 $EndComp
 $Comp
-L MOSFET:AO3402 M16
+L BMS-Board-rescue:AO3402-MOSFET M16
 U 1 1 5E9A140B
 P 12000 23100
+AR Path="/5E9A140B" Ref="M16"  Part="1"
+AR Path="/5E8E2BA1/5E9A140B" Ref="M16"  Part="1"
 F 0 "M16" H 12228 23146 50  0000 L CNN
 F 1 "AO3402" H 12228 23055 50  0000 L CNN
@@
 $EndComp
 $Comp
-L MOSFET:AO3402 M15
+L BMS-Board-rescue:AO3402-MOSFET M15
 U 1 1 5E9AA406
 P 12000 21900
+AR Path="/5E9AA406" Ref="M15"  Part="1"
+AR Path="/5E8E2BA1/5E9AA406" Ref="M15"  Part="1"
 F 0 "M15" H 12228 21946 50  0000 L CNN
 F 1 "AO3402" H 12228 21855 50  0000 L CNN
@@
 $EndComp
 $Comp
-L MOSFET:AO3402 M14
+L BMS-Board-rescue:AO3402-MOSFET M14
 U 1 1 5EA4749A
 P 12000 20700
+AR Path="/5EA4749A" Ref="M14"  Part="1"
+AR Path="/5E8E2BA1/5EA4749A" Ref="M14"  Part="1"
 F 0 "M14" H 12228 20746 50  0000 L CNN
 F 1 "AO3402" H 12228 20655 50  0000 L CNN
@@
 $EndComp
 $Comp
-L MOSFET:AO3402 M13
+L BMS-Board-rescue:AO3402-MOSFET M13
 U 1 1 5EA50EA1
 P 12000 19500
+AR Path="/5EA50EA1" Ref="M13"  Part="1"
+AR Path="/5E8E2BA1/5EA50EA1" Ref="M13"  Part="1"
 F 0 "M13" H 12228 19546 50  0000 L CNN
 F 1 "AO3402" H 12228 19455 50  0000 L CNN
@@
 $EndComp
 $Comp
-L MOSFET:AO3402 M12
+L BMS-Board-rescue:AO3402-MOSFET M12
 U 1 1 5EA59EF8
 P 12000 18300
+AR Path="/5EA59EF8" Ref="M12"  Part="1"
+AR Path="/5E8E2BA1/5EA59EF8" Ref="M12"  Part="1"
 F 0 "M12" H 12228 18346 50  0000 L CNN
 F 1 "AO3402" H 12228 18255 50  0000 L CNN
@@
 $EndComp
 $Comp
-L MOSFET:AO3402 M11
+L BMS-Board-rescue:AO3402-MOSFET M11
 U 1 1 5EA656B9
 P 12000 17100
+AR Path="/5EA656B9" Ref="M11"  Part="1"
+AR Path="/5E8E2BA1/5EA656B9" Ref="M11"  Part="1"
 F 0 "M11" H 12228 17146 50  0000 L CNN
 F 1 "AO3402" H 12228 17055 50  0000 L CNN
@@
 $EndComp
 $Comp
-L MOSFET:AO3402 M10
+L BMS-Board-rescue:AO3402-MOSFET M10
 U 1 1 5EA71F60
 P 12000 15900
+AR Path="/5EA71F60" Ref="M10"  Part="1"
+AR Path="/5E8E2BA1/5EA71F60" Ref="M10"  Part="1"
 F 0 "M10" H 12228 15946 50  0000 L CNN
 F 1 "AO3402" H 12228 15855 50  0000 L CNN
@@
 $EndComp
 $Comp
-L MOSFET:AO3402 M9
+L BMS-Board-rescue:AO3402-MOSFET M9
 U 1 1 5EAD0B07
 P 12000 14700
+AR Path="/5EAD0B07" Ref="M9"  Part="1"
+AR Path="/5E8E2BA1/5EAD0B07" Ref="M9"  Part="1"
 F 0 "M9" H 12228 14746 50  0000 L CNN
 F 1 "AO3402" H 12228 14655 50  0000 L CNN
@@
 $EndComp
 $Comp
-L MOSFET:AO3402 M8
+L BMS-Board-rescue:AO3402-MOSFET M8
 U 1 1 5EADCF0B
 P 12000 13500
+AR Path="/5EADCF0B" Ref="M8"  Part="1"
+AR Path="/5E8E2BA1/5EADCF0B" Ref="M8"  Part="1"
 F 0 "M8" H 12228 13546 50  0000 L CNN
 F 1 "AO3402" H 12228 13455 50  0000 L CNN
@@
 $EndComp
 $Comp
-L MOSFET:AO3402 M7
+L BMS-Board-rescue:AO3402-MOSFET M7
 U 1 1 5EAEAD35
 P 12000 12300
+AR Path="/5EAEAD35" Ref="M7"  Part="1"
+AR Path="/5E8E2BA1/5EAEAD35" Ref="M7"  Part="1"
 F 0 "M7" H 12228 12346 50  0000 L CNN
 F 1 "AO3402" H 12228 12255 50  0000 L CNN
@@
 $EndComp
 $Comp
-L MOSFET:AO3402 M6
+L BMS-Board-rescue:AO3402-MOSFET M6
 U 1 1 5EAFA213
 P 12000 11100
+AR Path="/5EAFA213" Ref="M6"  Part="1"
+AR Path="/5E8E2BA1/5EAFA213" Ref="M6"  Part="1"
 F 0 "M6" H 12228 11146 50  0000 L CNN
 F 1 "AO3402" H 12228 11055 50  0000 L CNN
@@
 $EndComp
 $Comp
-L MOSFET:AO3402 M5
+L BMS-Board-rescue:AO3402-MOSFET M5
 U 1 1 5EB0B2DF
 P 12000 9900
+AR Path="/5EB0B2DF" Ref="M5"  Part="1"
+AR Path="/5E8E2BA1/5EB0B2DF" Ref="M5"  Part="1"
 F 0 "M5" H 12228 9946 50  0000 L CNN
 F 1 "AO3402" H 12228 9855 50  0000 L CNN
@@
 $EndComp
 $Comp
-L MOSFET:AO3402 M4
+L BMS-Board-rescue:AO3402-MOSFET M4
 U 1 1 5EB21F8B
 P 12000 8700
+AR Path="/5EB21F8B" Ref="M4"  Part="1"
+AR Path="/5E8E2BA1/5EB21F8B" Ref="M4"  Part="1"
 F 0 "M4" H 12228 8746 50  0000 L CNN
 F 1 "AO3402" H 12228 8655 50  0000 L CNN
@@
 $EndComp
 $Comp
-L MOSFET:AO3402 M3
+L BMS-Board-rescue:AO3402-MOSFET M3
 U 1 1 5EBB1DCD
 P 12000 7500
+AR Path="/5EBB1DCD" Ref="M3"  Part="1"
+AR Path="/5E8E2BA1/5EBB1DCD" Ref="M3"  Part="1"
 F 0 "M3" H 12228 7546 50  0000 L CNN
 F 1 "AO3402" H 12228 7455 50  0000 L CNN
@@
 $EndComp
 $Comp
-L MOSFET:AO3402 M2
+L BMS-Board-rescue:AO3402-MOSFET M2
 U 1 1 5EBC9AD0
 P 12000 6300
+AR Path="/5EBC9AD0" Ref="M2"  Part="1"
+AR Path="/5E8E2BA1/5EBC9AD0" Ref="M2"  Part="1"
 F 0 "M2" H 12228 6346 50  0000 L CNN
 F 1 "AO3402" H 12228 6255 50  0000 L CNN
@@
 $EndComp
 $Comp
-L MOSFET:AO3402 M1
+L BMS-Board-rescue:AO3402-MOSFET M1
 U 1 1 5EBE32E1
 P 12000 5100
+AR Path="/5EBE32E1" Ref="M1"  Part="1"
+AR Path="/5E8E2BA1/5EBE32E1" Ref="M1"  Part="1"
 F 0 "M1" H 12228 5146 50  0000 L CNN
 F 1 "AO3402" H 12228 5055 50  0000 L CNN
